File: main_control_board.kicad_pcb (KiCad board)
At the start: 2 copper layers, 80 x 46 mm, 52 parts, among them J1 USB1/PWR IN, J10 GPIOs, J11 EXT_PWR, J12 PROG MODE, J2 USB_Out, J3 USB2/PWR IN, J4 USB_3, J5 USB_4, J6 I2C, J7 Display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

Commit message: update to latest
Parts:
- removed the C6 at (147.3, 100.7)
- moved R6 4.90 mm to (134.4, 98.0)
- moved R7 4.62 mm to (136.2, 98.0)
- moved R2 3.74 mm to (154.4, 118.5), turned to 180 degrees
- moved C3 2.17 mm to (151.8, 118.5)
- moved D6 0.59 mm to (151.6, 103.2)
- renumbered C7 to C6, U6 to U5
Connections:
- J10 pad 10: GPIO10 -> GPIO9
- J10 pad 12: GPIO11 -> GPIO10
- J10 pad 14: GND -> GPIO11
- J10 pad 4: GND -> VCC_5V
- J10 pad 6: GPIO8 -> GND
- J10 pad 8: GPIO9 -> GPIO8
- J6 pad 1: GND -> VCC_3V3
- J6 pad 2: VCC_3V3 -> GND
- J8 pad 3: POT/IO16 -> POT/IO18
- J8 pad 4: POT/IO15 -> POT/IO17
- U1 pad 19: POT/IO15 -> SDA
- U1 pad 20: POT/IO16 -> SCL
- U1 pad 21: SDA -> POT/IO17
- U1 pad 22: SCL -> POT/IO18
Routing:
- net POT/IO16: track 45.3 -> 0.00 mm, vias 1 -> 0
- net POT/IO15: track 43.7 -> 0.00 mm, vias 1 -> 0
- net POT/IO18: track 0.00 -> 43.0 mm, vias 0 -> 1
- net POT/IO17: track 0.00 -> 41.4 mm, vias 0 -> 1
- net GND: track 157.6 -> 150.6 mm, vias 17 -> 15
- net VCC_5V: track 115.8 -> 122.6 mm
- net Net-(U1-IO0): track 48.8 -> 52.6 mm
- net IR_RX: track 32.4 -> 28.9 mm
- net SDA: track 20.1 -> 23.6 mm, vias 2 -> 1
- net VCC_3V3: track 176.1 -> 173.4 mm
- net Net-(U4-Vs): track 5.70 -> 3.71 mm
- net SCL: track 22.7 -> 24.6 mm, vias 2 -> 1
- net BL/IO36: track 47.7 -> 46.3 mm
- net GPIO11: track 16.5 -> 17.6 mm
- net GPIO12: track 21.4 -> 20.5 mm
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Other:
- board text added: "3V3 GND POT/IO18 POT/IO17 CCW/IO46 CW/IO45"
- board text added: "3V3 GND SCL SDA"
- board text added: "5V 5V GND IO8 IO9 IO10 IO11 IO12 IO13 IO14"
- board text added: "GND BL/IO36 3V3 CLK/IO35 DIN/IO34 DC/IO33 CS/IO47 RST/IO26"
- board text removed: "3V3 GND POT/IO16 POT/IO15 CCW/IO46 CW/IO45"
- board text removed: "5V GND IO8 IO9 IO10 IO11 GND IO12 IO13 IO14"
- board text removed: "GND 3V3 SCL SDA"
- board text removed: "GND BL/IO35 3V3 CLK/IO36 DIN/IO34 DC/IO33 CS/IO26 RST/IO21"
