File: main_control_board.kicad_sch (KiCad schematic)
At the start: 49 parts, among them J1 USB1/PWR IN, J10 GPIOs, J11 EXT_PWR, J12 PROG MODE, J2 USB_Out, J3 USB2/PWR IN, J4 USB_3, J5 USB_4, J6 I2C, J7 Display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

Commit message: update to latest
Parts:
- removed C6: 10uF (NC), CL10A106KP8NNNC:CAPC1608X90N, symbol CL10A106KP8NNNC:CL10A106KP8NNNC
- renumbered C7 to C6, U6 to U5
Connections:
- net +3.3V: now also J6.1 (Pin_1); no longer J6.2 (Pin_2)
- net +5V: now also J10.4 (Pin_4)
- net GND: now also J10.6 (Pin_6), J6.2 (Pin_2); no longer J10.14 (Pin_14), J10.4 (Pin_4), J6.1 (Pin_1)
- net GPIO10: now also J10.12 (Pin_12); no longer J10.10 (Pin_10)
- net GPIO11: now also J10.14 (Pin_14); no longer J10.12 (Pin_12)
- net GPIO8: now also J10.8 (Pin_8); no longer J10.6 (Pin_6)
- net GPIO9: now also J10.10 (Pin_10); no longer J10.8 (Pin_8)
- net SCL: now also U1.20 (IO16); no longer U1.22 (IO18)
- net SDA: now also U1.19 (IO15); no longer U1.21 (IO17)
- net CS/IO47 renamed CS/IO27
- net POT/IO15 renamed POT/IO17
- net POT/IO17: now also U1.21 (IO17); no longer U1.19 (IO15)
- net POT/IO16 renamed POT/IO18
- net POT/IO18: now also U1.22 (IO18); no longer U1.20 (IO16)
Other:
- moved on the sheet: C6, D5, D6, J10, J11, J12, J2, J3, J4, J5, J6, J7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
